Commit message: some sketchy artifacts

File: config/panda.urdf (robot description, URDF)
Before this commit: robot panda_kinect, 16 links, 15 joints
Links:
- added link map
- added link panda_gripper
- added link sander
- link camera_base: geometry 
- link camera_body: geometry visual mesh filename=package://drone_panda/meshes/visual/kinect-model.stl
- link camera_visor: geometry 
- link ft_sensor_link: geometry collision mesh filename=package://drone_panda/meshes/force_torque_sensor.stl; visual mesh filename=package://drone_panda/meshes/force_torque_sensor.dae
- link panda_hand: geometry collision mesh filename=package://drone_panda/meshes/collision/hand.stl; visual mesh filename=package://drone_panda/meshes/visual/hand.dae
- link panda_leftfinger: geometry collision mesh filename=package://drone_panda/meshes/collision/finger.stl; visual mesh filename=package://drone_panda/meshes/visual/finger.dae
- link panda_link0: geometry collision mesh filename=package://drone_panda/meshes/collision/link0.stl; visual mesh filename=package://drone_panda/meshes/visual/link0.dae
- link panda_link1: geometry collision mesh filename=package://drone_panda/meshes/collision/link1.stl; visual mesh filename=package://drone_panda/meshes/visual/link1.dae
- link panda_link2: geometry collision mesh filename=package://drone_panda/meshes/collision/link2.stl; visual mesh filename=package://drone_panda/meshes/visual/link2.dae
- link panda_link3: geometry collision mesh filename=package://drone_panda/meshes/collision/link3.stl; visual mesh filename=package://drone_panda/meshes/visual/link3.dae
- link panda_link4: geometry collision mesh filename=package://drone_panda/meshes/collision/link4.stl; visual mesh filename=package://drone_panda/meshes/visual/link4.dae
- link panda_link5: geometry collision mesh filename=package://drone_panda/meshes/collision/link5.stl; visual mesh filename=package://drone_panda/meshes/visual/link5.dae
- link panda_link6: geometry collision mesh filename=package://drone_panda/meshes/collision/link6.stl; visual mesh filename=package://drone_panda/meshes/visual/link6.dae
- link panda_link7: geometry collision mesh filename=package://drone_panda/meshes/collision/link7.stl; visual mesh filename=package://drone_panda/meshes/visual/link7.dae
- link panda_rightfinger: geometry collision mesh filename=package://drone_panda/meshes/collision/finger.stl; visual mesh filename=package://drone_panda/meshes/visual/finger.dae
Joints:
- added joint panda_base_map: type fixed, parent panda_link0, child map, origin xyz=0 0 0.0 rpy=0 0 0, axis 0 0 0
- added joint panda_gripper_joint: type fixed, parent panda_link8, child panda_gripper, origin xyz=-0.000 -0.000 0.103 rpy=3.1416 0.000 -0.785, axis 0 0 0
- added joint sander_joint: type fixed, parent panda_link8, child sander, origin xyz=-0.000 -0.000 0.144 rpy=3.1416 0.000 -0.785, axis 0 0 0
- joint fake_base: origin xyz=0.156 -0.041 0.00 rpy=-1.586 0.010 -1.585 -> xyz=0.08211274 0.0 0.00823 rpy=3.14 -1.57 0.0; parent panda_link6 -> panda_hand
- joint panda_joint4: limit lower=-3.0718 upper=-0.2698 effort=87 velocity=2.1750 -> lower=-3.0718 upper=-0.1698 effort=87 velocity=2.1750

Commit message: Updated to avoid resonances

File: config/panda.urdf (robot description, URDF)
Before this commit: robot panda_kinect, 19 links, 18 joints
Joints:
- joint panda_joint4: limit lower=-3.0718 upper=-0.1698 effort=87 velocity=2.1750 -> lower=-3.0718 upper=-0.3698 effort=87 velocity=2.1750
